File: hw1/shematic.kicad_pcb (KiCad board)
At the start: 2 copper layers, 26 parts, among them J1 Conn_01x02_Pin, J2 Conn_01x04_Pin, SW1 SW_MEC_5G, U1 AMS1117-3.3, U2 STM32F411CEUx

Commit message: hw2 shema update
Parts:
- C2: value 10n -> 0.01u
- C9: footprint Capacitor_SMD:C_1812_4532Metric_Pad1.57x3.40mm_HandSolder -> Capacitor_SMD:C_1206_3216Metric_Pad1.33x1.80mm_HandSolder
- JP1: footprint Connector_PinHeader_2.54mm:PinHeader_1x02_P2.54mm_Horizontal -> Connector_PinHeader_1.00mm:PinHeader_1x02_P1.00mm_Vertical
- U2: value STM32F411CEUx -> STM32F103C8Tx; footprint Package_DFN_QFN:QFN-48-1EP_7x7mm_P0.5mm_EP5.6x5.6mm -> Package_QFP:LQFP-48_7x7mm_P0.5mm
- moved C7 66.1 mm to (148.9, 85.7)
- moved C8 66.1 mm to (148.9, 89.1)
- moved C6 56.7 mm to (140.8, 76.6), turned to -90 degrees
- moved C1 46.0 mm to (126.4, 74.9), turned to -90 degrees
- moved J2 44.4 mm to (149.9, 74.3), turned to 180 degrees
- moved JP1 42.5 mm to (132.7, 68.6), turned to 90 degrees
- moved U2 40.8 mm to (134.2, 77.2)
- moved D5 34.9 mm to (147.0, 69.2), turned to 180 degrees
- moved D6 34.8 mm to (147.0, 71.8), turned to 180 degrees
- moved R3 34.0 mm to (137.8, 68.6), turned to 180 degrees
- moved SW1 26.4 mm to (116.7, 71.7)
- moved C5 20.4 mm to (127.6, 87.6)
- moved C9 19.2 mm to (127.8, 80.6), turned to -90 degrees
- moved J1 16.5 mm to (94.6, 70.5), turned to 180 degrees
- moved D3 15.6 mm to (108.0, 65.4)
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Connections:
- C10 pad 2: Net-(U2-VCAP1) -> unconnected-(C10-Pad2)
- C5 pad 2: Net-(C5-Pad2) -> GND
- C6 pad 2: Net-(C5-Pad2) -> GND
- C7 pad 2: Net-(C5-Pad2) -> GND
- C8 pad 2: Net-(C5-Pad2) -> GND
- C9 pad 2: Net-(C5-Pad2) -> GND
- SW1 pad 2: GND -> Net-(D2-A)
- U2 pad 22: Net-(U2-VCAP1) -> unconnected-(U2-PB11-Pad22)
