File: hw1/shematic.kicad_sch (KiCad schematic)
At the start: 26 parts, among them J1 Conn_01x02_Pin, J2 Conn_01x04_Pin, SW1 SW_MEC_5G, U1 AMS1117-3.3, U2 STM32F411CEUx

Commit message: hw2 shema update
Parts:
- removed U2: STM32F411CEUx, Package_DFN_QFN:QFN-48-1EP_7x7mm_P0.5mm_EP5.6x5.6mm, symbol MCU_ST_STM32F4:STM32F411CEUx
- added U2: STM32F103C8Tx, Package_QFP:LQFP-48_7x7mm_P0.5mm, symbol MCU_ST_STM32F1:STM32F103C8Tx
- C2: value 10n -> 0.01u
- C9: footprint Capacitor_SMD:C_1812_4532Metric_Pad1.57x3.40mm_HandSolder -> Capacitor_SMD:C_1206_3216Metric_Pad1.33x1.80mm_HandSolder
Connections:
- net +3.3V: now also U2.1 (VBAT), U2.24 (VDD), U2.36 (VDD), U2.48 (VDD), U2.9 (VDDA)
- net GND: now also C5.2, C6.2, C7.2, C8.2, C9.2, U2.23 (VSS), U2.35 (VSS), U2.47 (VSS), U2.8 (VSSA)
- net at C1.2, D2.2 (A), R1.1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: now also U2.7 (NRST)
- net at R4.1: now also U2.2 (PC13)
- net at D5.1 (K), J2.3 (Pin_3): now also U2.34 (PA13)
- net at D6.1 (K), J2.2 (Pin_2): now also U2.37 (PA14)
- net at JP1.2 (B), R3.2: now also U2.44 (BOOT0)
- no-connect marks 33 -> 35
Other:
- moved on the sheet: C10
